File: Hardware/_autosave-Bast_WAN.sch (KiCad schematic (older format))
At the start: 34 parts, among them J1 USB_B_Micro, J2 Conn_Right, J3 Conn_Left, J4 Conn_Battery, J5 Conn_ARM_JTAG_SWD_10, Q1 DMG3415U-7, SW1 RST, U1 RAK4260, U2 AP2112K-3.3TRG1, U3 ATECC608A-TNGLORA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

Commit message: add swd standard connector
Parts:
- J5: footprint (none) -> Connector_PinHeader_1.27mm:PinHeader_2x05_P1.27mm_Vertical
Changed lines of the file:
@@
 F 0 "J5" H 9850 5645 50  0000 R CNN
 F 1 "Conn_ARM_JTAG_SWD_10" V 9685 5515 50  0000 R CNN
-F 2 "" H 10145 5105 50  0001 C CNN
+F 2 "Connector_PinHeader_1.27mm:PinHeader_2x05_P1.27mm_Vertical" H 10145 5105 50  0001 C CNN
 F 3 "http://infocenter.arm.com/help/topic/com.arm.doc.ddi0314h/DDI0314H_coresight_components_trm.pdf" V 9795 3855 50  0001 C CNN
 	1    10145 5105
