File: Hardware/Bast_WAN.kicad_sch (KiCad schematic)
At the start: 30 parts

Commit message: Fix GND for AREF and Extra pin
Thanks Kongduino
Parts:
- removed D1: (no value), symbol Bast_WAN-rescue:D_TVS_ALT-Device
- added D1: PGB1010402KR, Diode_THT:D_DO-201AE_P15.24mm_Horizontal, symbol Diode:1N62xxCA
- AE1: value (none) -> Antenna; footprint (none) -> bast-wan:SMA_EDGE
- C1: value (none) -> 0.1uF; footprint (none) -> Capacitor_SMD:C_0603_1608Metric_Pad1.05x0.95mm_HandSolder
- C2: value (none) -> 47pF; footprint (none) -> Capacitor_SMD:C_0603_1608Metric_Pad1.05x0.95mm_HandSolder
- C3, C4, C5: value (none) -> 10uF; footprint (none) -> Capacitor_SMD:C_0603_1608Metric_Pad1.05x0.95mm_HandSolder
- D2: value (none) -> MBR120; footprint (none) -> Diode_SMD:D_SOD-123
- D4: value (none) -> CHR; footprint (none) -> LED_SMD:LED_0805_2012Metric_Pad1.15x1.40mm_HandSolder
- D5: value (none) -> D13; footprint (none) -> LED_SMD:LED_0805_2012Metric_Pad1.15x1.40mm_HandSolder
- J1: value (none) -> USB_B_Micro; footprint (none) -> Connectors:U254051N4BH806
- J2: value (none) -> Conn_Right; footprint (none) -> Connector_PinSocket_2.54mm:PinSocket_1x12_P2.54mm_Vertical
- J3: value (none) -> Conn_Left; footprint (none) -> Connector_PinSocket_2.54mm:PinSocket_1x16_P2.54mm_Vertical
- J4: value (none) -> Conn_Battery; footprint (none) -> bast-wan:JST_S2B-PH-SM4-TB(LF)(SN)
- J5: value (none) -> SWD; footprint (none) -> Connector_PinHeader_2.54mm:PinHeader_1x04_P2.54mm_Vertical
- Q1: value (none) -> DMG3415U-7; footprint (none) -> Package_TO_SOT_SMD:SOT-23
- R1, R2: value (none) -> 100K; footprint (none) -> Resistor_SMD:R_0603_1608Metric_Pad1.05x0.95mm_HandSolder
- R10, R11: value (none) -> 10K; footprint (none) -> Resistor_SMD:R_0603_1608Metric_Pad1.05x0.95mm_HandSolder
- R3: value (none) -> 1M; footprint (none) -> Resistor_SMD:R_0603_1608Metric_Pad1.05x0.95mm_HandSolder
- R4: value (none) -> 1.5M; footprint (none) -> Resistor_SMD:R_0603_1608Metric_Pad1.05x0.95mm_HandSolder
- R6: value (none) -> 4.7K; footprint (none) -> Resistor_SMD:R_0603_1608Metric_Pad1.05x0.95mm_HandSolder
- R8, R9: value (none) -> 330; footprint (none) -> Resistor_SMD:R_0603_1608Metric_Pad1.05x0.95mm_HandSolder
- SW1: value (none) -> RST; footprint (none) -> Button_Switch_SMD:SW_SPST_TL3342
- U1: value (none) -> RAK4260; footprint (none) -> bast-wan:RAK4260-footprint_w_solder_paste
- U2: value (none) -> AP2112K-3.3TRG1; footprint (none) -> Package_TO_SOT_SMD:TSOT-23-5
- U3: value (none) -> ATECC608A-TNGLORA; footprint (none) -> Package_DFN_QFN:DFN-8-1EP_3x2mm_P0.5mm_EP1.3x1.5mm
- U5: value (none) -> MCP73831-3-OT; footprint (none) -> Package_TO_SOT_SMD:SOT-23-5
Connections:
- net ANT: now also D1.2 (A2)
- net GND: now also D1.1 (A1); no longer J3.16 (Pin_16), J3.3 (Pin_3)
- no-connect marks 1 -> 3
